File: ev_charger.kicad_pcb (KiCad board)
At the start: 2 copper layers, 54.2 x 34.8 mm, 33 parts, among them J1 Conn_01x03, J2 Conn_01x02, J3 Conn_01x02, J4 Conn_01x04, J5 Conn_01x02, J6 Conn_01x02, J7 Conn_01x02, J8 Conn_01x02, J9 Conn_01x02, U1 TPS61040DBV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

Commit message: Fix missing via bug
Routing:
- net GND: vias 11 -> 16
Other:
- board text added: "Rev. 0.1.1"
- board text added: "VDD"
- board text removed: "3.3V"
- board text removed: "Rev. 0.1.0"
Changed lines of the file:
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@@
 		)
 	)
-	(gr_text "3.3V"
+	(gr_text "VDD"
 		(at 81.75 83.5 90)
 		(layer "F.SilkS")
@@
 		)
 	)
-	(gr_text "Rev. 0.1.0"
+	(gr_text "Rev. 0.1.1"
 		(at 71.25 85.5 0)
 		(layer "F.SilkS")
@@
 	)
 	(via
+		(at 96.2 65.4)
+		(size 0.6)
+		(drill 0.3)
+		(layers "F.Cu" "B.Cu")
+		(free yes)
+		(net 1)
+	)
+	(via
 		(at 102 62)
 		(size 0.6)
@@
 	)
 	(via
+		(at 91.4 74.4)
+		(size 0.6)
+		(drill 0.3)
+		(layers "F.Cu" "B.Cu")
+		(free yes)
+		(net 1)
+	)
+	(via
 		(at 79.25 65.25)
 		(size 0.6)
@@
 	)
 	(via
+		(at 96.2 74.4)
+		(size 0.6)
+		(drill 0.3)
+		(layers "F.Cu" "B.Cu")
+		(free yes)
+		(net 1)
+	)
+	(via
+		(at 80.2 74.8)
+		(size 0.6)
+		(drill 0.3)
+		(layers "F.Cu" "B.Cu")
+		(free yes)
+		(net 1)
+	)
+	(via
 		(at 76.2 69.4)
 		(size 0.6)
 		(drill 0.3)
+		(layers "F.Cu" "B.Cu")
+		(free yes)
+		(net 1)
+	)
+	(via
+		(at 91.6 65.4)
+		(size 0.6)
+		(drill 0.3)

Commit message: Rename 3.3v to 3v/VDD
Connections:
- net +3.3V renamed 3V
Changed lines of the file:
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@@
 	(net 4 "/PWM_OUT")
 	(net 5 "/PWM_IN")
-	(net 6 "+3.3V")
+	(net 6 "3V")
 	(net 7 "/PILOT_SENSE")
 	(net 8 "Net-(D1-K)")
@@
 			(layers "F.Cu" "F.Mask" "F.Paste")
 			(roundrect_rratio 0.25)
-			(net 6 "+3.3V")
+			(net 6 "3V")
 			(pintype "passive")
 		)
@@
 			(layers "F.Cu" "F.Mask" "F.Paste")
 			(roundrect_rratio 0.25)
-			(net 6 "+3.3V")
+			(net 6 "3V")
 			(pinfunction "EN")
 			(pintype "input")
@@
 			(layers "F.Cu" "F.Mask" "F.Paste")
 			(roundrect_rratio 0.25)
-			(net 6 "+3.3V")
+			(net 6 "3V")
 			(pinfunction "VIN")
 			(pintype "power_in")
@@
 			(layers "*.Cu" "*.Mask")
 			(remove_unused_layers no)
-			(net 6 "+3.3V")
+			(net 6 "3V")
 			(pinfunction "Pin_1")
 			(pintype "passive")
@@
 			(layers "F.Cu" "F.Mask" "F.Paste")
 			(roundrect_rratio 0.222222)
-			(net 6 "+3.3V")
+			(net 6 "3V")
 			(pinfunction "1")
 			(pintype "passive")
@@
 			(layers "F.Cu" "F.Mask" "F.Paste")
 			(roundrect_rratio 0.25)
-			(net 6 "+3.3V")
+			(net 6 "3V")
 			(pintype "passive")
 		)
@@
 			(layers "F.Cu" "F.Mask" "F.Paste")
 			(roundrect_rratio 0.25)
-			(net 6 "+3.3V")
+			(net 6 "3V")
 			(pintype "passive")
 		)

Commit message: Adjust resistor values
- Change r3 to 1k to adjust output CE PWM voltage.
- Change r4 to 46k to increase bias. This avoids negative sense
  voltages.
Parts:
- R3: value 560R -> 1k
- R4: value 56k -> 47k
Changed lines of the file:
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@@
 			)
 		)
-		(property "Value" "56k"
+		(property "Value" "47k"
 			(at 0 1.43 0)
 			(layer "F.Fab")
@@
 			)
 		)
-		(property "LCSC" "C23206"
+		(property "LCSC" "C25819"
 			(at 0 0 0)
 			(unlocked yes)
@@
 			)
 		)
-		(property "Value" "560R"
+		(property "Value" "1k"
 			(at 0 1.43 0)
 			(layer "F.Fab")
@@
 			)
 		)
-		(property "LCSC" "C23204"
+		(property "LCSC" "C21190"
 			(at 0 0 0)
 			(unlocked yes)
